File: project/eagle/DC_bias_circuit/DC_bias_circuit.brd (EAGLE design)
At the start: 30.1 x 15.2 mm, 17 parts, among them Q1 MMBT3906LT1SMD, Q2 MMBT3906LT1SMD, Q3 SAV-541+

Commit message: created tappered TL
Connections:
- net N$7 renamed GATE
- net N$8 renamed DRAIN
Changed lines of the file:
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@@
 <?xml version="1.0" encoding="utf-8"?>
 <!DOCTYPE eagle SYSTEM "eagle.dtd">
-<eagle version="7.5.0">
+<eagle version="6.5.0">
 <drawing>
 <settings>
@@
 <pass name="Default">
 <param name="RoutingGrid" value="50mil"/>
-<param name="AutoGrid" value="1"/>
-<param name="Efforts" value="0"/>
-<param name="TopRouterVariant" value="1"/>
 <param name="tpViaShape" value="round"/>
 <param name="PrefDir.1" value="|"/>
@@
 <wire x1="11.43" y1="8.89" x2="12.3825" y2="9.8425" width="0.4064" layer="1"/>
 </signal>
-<signal name="N$7">
+<signal name="GATE">
 <contactref element="L1" pad="2"/>
 <contactref element="Q3" pad="3"/>
@@
 <wire x1="14.9225" y1="2.8575" x2="14.9225" y2="5.2675" width="0.4064" layer="1"/>
 </signal>
-<signal name="N$8">
+<signal name="DRAIN">
 <contactref element="R5" pad="2"/>
 <contactref element="Q3" pad="1"/>
