File: project/eagle/DC_bias_circuit/DC_bias_circuit.sch (EAGLE design)
At the start: 17 parts, among them Q1 MMBT3906LT1SMD, Q2 MMBT3906LT1SMD, Q3 SAV-541+

Commit message: created tappered TL
Connections:
- net N$7 renamed GATE
- net N$8 renamed DRAIN
Changed lines of the file:
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@@
 </segment>
 </net>
-<net name="N$7" class="0">
+<net name="GATE" class="0">
 <segment>
 <pinref part="L1" gate="G$1" pin="2"/>
@@
 </segment>
 </net>
-<net name="N$8" class="0">
+<net name="DRAIN" class="0">
 <segment>
 <pinref part="R5" gate="G$1" pin="2"/>
