File: project/eagle/LNA/version1/LNA_V1.brd (EAGLE design)
At the start: 34.4 x 45.7 mm, 21 parts, among them Q1 MMBT3906LT1SMD, Q2 MMBT3906LT1SMD, Q3 SAV-541+, X1 SMA-142-0701-871/876, X2 SMA-142-0701-871/876

Commit message: updated lna board
Connections:
- net N$2 renamed VG
- net N$6 renamed VD
Changed lines of the file:
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@@
 <wire x1="17.65" y1="31.95" x2="20.46" y2="29.04" width="0.3" layer="1"/>
 </signal>
-<signal name="N$2">
+<signal name="VG">
 <contactref element="Q2" pad="C"/>
 <contactref element="R4" pad="1"/>
@@
 <wire x1="27.47" y1="26.5" x2="27.5" y2="26.47" width="0.5" layer="1"/>
 </signal>
-<signal name="N$6">
+<signal name="VD">
 <contactref element="R2" pad="1"/>
 <contactref element="Q2" pad="E"/>
