File: project/eagle/LNA/version1/LNA_V1.sch (EAGLE design)
At the start: 21 parts, among them Q1 MMBT3906LT1SMD, Q2 MMBT3906LT1SMD, Q3 SAV-541+, X1 SMA-142-0701-871/876, X2 SMA-142-0701-871/876

Commit message: updated lna board
Connections:
- net N$2 renamed VG
- net N$6 renamed VD
Changed lines of the file:
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@@
 <?xml version="1.0" encoding="utf-8"?>
 <!DOCTYPE eagle SYSTEM "eagle.dtd">
-<eagle version="6.5.0">
+<eagle version="7.5.0">
 <drawing>
 <settings>
@@
 </segment>
 </net>
-<net name="N$2" class="0">
+<net name="VG" class="0">
 <segment>
 <pinref part="Q2" gate="G$1" pin="C"/>
@@
 </segment>
 </net>
-<net name="N$6" class="0">
+<net name="VD" class="0">
 <segment>
 <pinref part="R2" gate="G$1" pin="1"/>
