File: project/eagle/LNA/cameron_v1/LNA_V1.brd (EAGLE design)
At the start: 50 x 45.8 mm, 14 parts, among them Q1 MMBT3906LT1SMD, Q2 MMBT3906LT1SMD, Q3 SAV-541+, X1 SMA-142-0701-871/876, X2 SMA-142-0701-871/876

Commit message: added stabilizing resistors
Parts:
- added R5: 50, rcl:M1206
- added R6: 100, rcl:M1206
Connections:
- net GND: now also R5.2, R6.2
- net INPUT: now also R5.1
- net OUTPUT: now also R6.1
Routing:
- net INPUT: track 0.00 -> 3.49 mm
- net OUTPUT: track 0.00 -> 3.48 mm
- net GND: track 5.11 -> 7.58 mm, vias 4 -> 6
Changed lines of the file:
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@@
 <setting verticaltext="up"/>
 </settings>
-<grid distance="10" unitdist="mil" unit="mil" style="lines" multiple="1" display="yes" altdistance="0.025" altunitdist="inch" altunit="inch"/>
+<grid distance="0.003125" unitdist="mic" unit="mil" style="lines" multiple="1" display="yes" altdistance="0.025" altunitdist="inch" altunit="inch"/>
 <layers>
 <layer number="1" name="Top" color="4" fill="1" visible="yes" active="yes"/>
@@
 <attribute name="NAME" x="49.138321875" y="2.708153125" size="1.778" layer="25" rot="R180"/>
 </element>
+<element name="R5" library="rcl" package="M1206" value="50" x="15.372421875" y="7.241984375" rot="R270"/>
+<element name="R6" library="rcl" package="M1206" value="100" x="24.689553125" y="5.923" rot="R270"/>
 </elements>
 <signals>
@@
 <wire x1="19.649846875" y1="25.89825625" x2="19.720153125" y2="25.82795" width="0.4064" layer="1"/>
 <wire x1="25.745846875" y1="27.29195" x2="25.745846875" y2="25.82795" width="0.4064" layer="1"/>
+<via x="15.3887375" y="4.604246875" extent="1-16" drill="0.4"/>
+<via x="24.74955" y="3.315909375" extent="1-16" drill="0.4"/>
+<contactref element="R5" pad="2"/>
+<contactref element="R6" pad="2"/>
+<wire x1="15.372421875" y1="5.841984375" x2="15.372421875" y2="4.6205625" width="0.4064" layer="1"/>
+<wire x1="15.372421875" y1="4.6205625" x2="15.3887375" y2="4.604246875" width="0.4064" layer="1"/>
+<wire x1="24.689553125" y1="4.523" x2="24.689553125" y2="3.37590625" width="0.4064" layer="1"/>
+<wire x1="24.689553125" y1="3.37590625" x2="24.74955" y2="3.315909375" width="0.4064" layer="1"/>
 <wire x1="47.207921875" y1="13.477753125" x2="47.207921875" y2="13.477753125" width="0" layer="19" extent="1-16"/>
 <wire x1="47.207921875" y1="4.638553125" x2="47.207921875" y2="4.638553125" width="0" layer="19" extent="1-16"/>
@@
 <vertex x="18.93950625" y="10.097296875"/>
 </polygon>
+<contactref element="R5" pad="1"/>
+<wire x1="15.298715625" y1="12.07604375" x2="15.298715625" y2="8.8088875" width="0.4064" layer="1"/>
+<wire x1="15.298715625" y1="8.8088875" x2="15.456546875" y2="8.65105625" width="0.4064" layer="1"/>
 </signal>
 <signal name="ISO_INPUT">
@@
 <vertex x="21.128334375" y="9.304184375"/>
 </polygon>
+<contactref element="R6" pad="1"/>
+<wire x1="24.77925" y1="10.764640625" x2="24.77925" y2="7.412696875" width="0.4064" layer="1"/>
+<wire x1="24.77925" y1="7.412696875" x2="24.689553125" y2="7.323" width="0.4064" layer="1"/>
 </signal>
 <signal name="ISO_OUTPUT">
