File: project/FSK/eagle/splitter/splitter.brd (EAGLE design)
At the start: 100 x 80 mm, 4 parts, among them X1 SMA-142-0701-801/806, X2 SMA-142-0701-801/806, X3 SMA-142-0701-801/806

Commit message: created test board for diode
Other:
- board size 100 x 80 mm -> 39.1 x 34.2 mm
Changed lines of the file:
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@@
 <setting verticaltext="up"/>
 </settings>
-<grid distance="0.002" unitdist="mm" unit="mm" style="lines" multiple="1" display="no" altdistance="0.025" altunitdist="inch" altunit="inch"/>
+<grid distance="0.003125" unitdist="mic" unit="mm" style="lines" multiple="1" display="no" altdistance="0.025" altunitdist="inch" altunit="inch"/>
 <layers>
 <layer number="1" name="Top" color="4" fill="1" visible="yes" active="yes"/>
@@
 <board>
 <plain>
-<wire x1="0" y1="0" x2="100" y2="0" width="0" layer="20"/>
-<wire x1="100" y1="0" x2="100" y2="80" width="0" layer="20"/>
-<wire x1="100" y1="80" x2="0" y2="80" width="0" layer="20"/>
-<wire x1="0" y1="80" x2="0" y2="0" width="0" layer="20"/>
+<wire x1="5.6" y1="10.4" x2="44.7" y2="10.4" width="0" layer="20"/>
+<wire x1="44.7" y1="10.4" x2="44.7" y2="44.6" width="0" layer="20"/>
+<wire x1="44.7" y1="44.6" x2="5.6" y2="44.6" width="0" layer="20"/>
+<wire x1="5.6" y1="44.6" x2="5.6" y2="10.4" width="0" layer="20"/>
+<rectangle x1="38.628475" y1="36.04445" x2="39.728540625" y2="39.53508125" layer="1"/>
 </plain>
 <attributes>
@@
 <vertex x="37.452" y="37.816"/>
 </polygon>
-<wire x1="42.1386" y1="37.799909375" x2="38.499284375" y2="37.799909375" width="3.3" layer="1"/>
 <wire x1="42.1386" y1="37.799909375" x2="42.1386" y2="37.846" width="0.05" layer="1"/>
 <polygon width="0.05" layer="1">
@@
 <vertex x="34.7" y="34.854"/>
 </polygon>
+<wire x1="38.499284375" y1="37.799909375" x2="42.1386" y2="37.799909375" width="0.01" layer="1"/>
 </signal>
 <signal name="O3">
