File: project/FSK/eagle/LNA/LNA.sch (EAGLE design)
At the start: 9 parts, among them X1 SMA-142-0711-821/826, X2 SMA-142-0711-821/826, X3 22-23-2021

Commit message: changed traces on the LNA board to be 500 ohm, started FSK schematic
Connections:
- net N$4 renamed D_OUT
- net N$5 renamed D_IN
Changed lines of the file:
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@@
 </segment>
 </net>
-<net name="N$4" class="0">
+<net name="D_OUT" class="0">
 <segment>
 <pinref part="C4" gate="G$1" pin="2"/>
@@
 </segment>
 </net>
-<net name="N$5" class="0">
+<net name="D_IN" class="0">
 <segment>
 <pinref part="X1" gate="G1" pin="1"/>
