File: project/FSK/eagle/LNA/LNA.sch (EAGLE design)
At the start: 9 parts, among them X1 SMA-142-0711-821/826, X2 SMA-142-0711-821/826, X3 22-23-2021

Commit message: added schematic for 7segment driver
Parts:
- added IN1, OUT2: TEE_TL1, ECE532_Parts:TEE_TL1
Connections:
- removed net D_IN: C1.1, X1.1
- removed net D_OUT: C4.2, X2.1
- new net IN1: C1.1, IN1.T_B, IN1.T_L, IN1.T_R, X1.1
- new net OUT2: C4.2, OUT2.T_B, OUT2.T_L, OUT2.T_R, X2.1
Other:
- moved on the sheet: X1, X2
Changed lines of the file:
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@@
 <?xml version="1.0" encoding="utf-8"?>
 <!DOCTYPE eagle SYSTEM "eagle.dtd">
-<eagle version="7.5.0">
+<eagle version="6.5.0">
 <drawing>
 <settings>
@@
 <part name="SUPPLY7" library="supply2" deviceset="AGND" device=""/>
 <part name="L1" library="resistor" deviceset="L-US" device="L3230M" value="820nH"/>
+<part name="IN1" library="ECE532_Parts" deviceset="TEE_TL1" device=""/>
+<part name="OUT2" library="ECE532_Parts" deviceset="TEE_TL1" device=""/>
 </parts>
 <sheets>
@@
 <instance part="SUPPLY4" gate="G$1" x="73.66" y="68.58"/>
 <instance part="C4" gate="G$1" x="121.92" y="53.34" rot="R90"/>
-<instance part="X1" gate="G1" x="38.1" y="53.34"/>
-<instance part="X2" gate="G1" x="137.16" y="53.34" rot="MR0"/>
-<instance part="SUPPLY5" gate="G$1" x="40.64" y="45.72"/>
-<instance part="SUPPLY6" gate="G$1" x="132.08" y="45.72"/>
+<instance part="X1" gate="G1" x="22.86" y="53.34" smashed="yes">
+<attribute name="NAME" x="20.32" y="56.642" size="1.778" layer="95"/>
+</instance>
+<instance part="X2" gate="G1" x="152.4" y="53.34" smashed="yes" rot="MR0">
+<attribute name="NAME" x="154.94" y="56.642" size="1.778" layer="95" rot="MR0"/>
+</instance>
+<instance part="SUPPLY5" gate="G$1" x="25.4" y="45.72"/>
+<instance part="SUPPLY6" gate="G$1" x="149.86" y="45.72"/>
 <instance part="X3" gate="-1" x="76.2" y="93.98" rot="R90"/>
 <instance part="X3" gate="-2" x="78.74" y="93.98" rot="R90"/>
 <instance part="SUPPLY7" gate="G$1" x="76.2" y="83.82"/>
 <instance part="L1" gate="G$1" x="114.3" y="76.2"/>
+<instance part="IN1" gate="G$1" x="35.56" y="53.34"/>
+<instance part="OUT2" gate="G$1" x="137.16" y="53.34"/>
 </instances>
 <busses>
@@
 <segment>
 <pinref part="SUPPLY6" gate="G$1" pin="AGND"/>
-<wire x1="132.08" y1="48.26" x2="132.08" y2="50.8" width="0.1524" layer="91"/>
+<wire x1="149.86" y1="48.26" x2="149.86" y2="50.8" width="0.1524" layer="91"/>
 <pinref part="X2" gate="G1" pin="2"/>
-<wire x1="132.08" y1="50.8" x2="134.62" y2="50.8" width="0.1524" layer="91"/>
 </segment>
 <segment>
 <pinref part="X1" gate="G1" pin="2"/>
 <pinref part="SUPPLY5" gate="G$1" pin="AGND"/>
-<wire x1="40.64" y1="50.8" x2="40.64" y2="48.26" width="0.1524" layer="91"/>
+<wire x1="25.4" y1="50.8" x2="25.4" y2="48.26" width="0.1524" layer="91"/>
 </segment>
 <segment>
@@
 </segment>
 </net>
+<net name="IN1" class="0">
+<segment>
+<pinref part="X1" gate="G1" pin="1"/>
+<pinref part="IN1" gate="G$1" pin="T_L"/>
+<wire x1="25.4" y1="53.34" x2="27.94" y2="53.34" width="0.1524" layer="91"/>
+<wire x1="27.94" y1="53.34" x2="27.94" y2="45.72" width="0.1524" layer="91"/>
+<pinref part="IN1" gate="G$1" pin="T_R"/>
+<pinref part="C1" gate="G$1" pin="1"/>
+<wire x1="43.18" y1="53.34" x2="45.72" y2="53.34" width="0.1524" layer="91"/>
+<pinref part="IN1" gate="G$1" pin="T_B"/>
+<wire x1="35.56" y1="45.72" x2="45.72" y2="45.72" width="0.1524" layer="91"/>
+<wire x1="45.72" y1="45.72" x2="45.72" y2="53.34" width="0.1524" layer="91"/>
+<wire x1="27.94" y1="45.72" x2="35.56" y2="45.72" width="0.1524" layer="91"/>
+<junction x="45.72" y="53.34"/>
+<junction x="35.56" y="45.72"/>
+<junction x="27.94" y="53.34"/>
+</segment>
+</net>
+<net name="OUT2" class="0">
+<segment>
+<pinref part="C4" gate="G$1" pin="2"/>
+<pinref part="OUT2" gate="G$1" pin="T_L"/>
+<wire x1="127" y1="53.34" x2="129.54" y2="53.34" width="0.1524" layer="91"/>
+<pinref part="OUT2" gate="G$1" pin="T_B"/>
+<wire x1="137.16" y1="45.72" x2="127" y2="45.72" width="0.1524" layer="91"/>
+<wire x1="127" y1="45.72" x2="127" y2="53.34" width="0.1524" layer="91"/>
+<wire x1="137.16" y1="45.72" x2="147.32" y2="45.72" width="0.1524" layer="91"/>
+<wire x1="147.32" y1="45.72" x2="147.32" y2="53.34" width="0.1524" layer="91"/>
+<pinref part="OUT2" gate="G$1" pin="T_R"/>
+<pinref part="X2" gate="G1" pin="1"/>
+<wire x1="144.78" y1="53.34" x2="147.32" y2="53.34" width="0.1524" layer="91"/>
+<junction x="147.32" y="53.34"/>
+<wire x1="147.32" y1="53.34" x2="149.86" y2="53.34" width="0.1524" layer="91"/>
+<junction x="127" y="53.34"/>
+</segment>
+</net>
 <net name="IN" class="0">
 <segment>
@@
 </segment>
 </net>
-<net name="D_OUT" class="0">
-<segment>
-<pinref part="C4" gate="G$1" pin="2"/>
-<pinref part="X2" gate="G1" pin="1"/>
-<wire x1="127" y1="53.34" x2="134.62" y2="53.34" width="0.1524" layer="91"/>
-</segment>
-</net>
-<net name="D_IN" class="0">
-<segment>
-<pinref part="X1" gate="G1" pin="1"/>
-<pinref part="C1" gate="G$1" pin="1"/>
-<wire x1="40.64" y1="53.34" x2="45.72" y2="53.34" width="0.1524" layer="91"/>
-</segment>
-</net>
