File: project/FSK/eagle/LNA/LNA.brd (EAGLE design)
At the start: 40.2 x 23.2 mm, 9 parts, among them X1 SMA-142-0711-821/826, X2 SMA-142-0711-821/826, X3 22-23-2021

Commit message: added schematic for 7segment driver
Parts:
- added IN1, OUT2: TEE_TL1, ECE532_Parts:TEE_TL1
- moved X2 24.7 mm to (94.0, 24.8)
- moved X1 21.0 mm to (8.13, 29.0)
Connections:
- removed net D_IN: C1.1, X1.1
- removed net D_OUT: C4.2, X2.1
- new net IN1: C1.1, IN1.T_B, IN1.T_L, IN1.T_R, X1.1
- new net OUT2: C4.2, OUT2.T_B, OUT2.T_L, OUT2.T_R, X2.1
Routing:
- added copper zone on layer 1, net OUT2
- added copper zone on layer 1, net XX
- removed copper zone on layer 16, net AGND
- removed copper zone on layer 1, net D_IN
- removed copper zone on layer 1, net D_OUT
Other:
- board size 40.2 x 23.2 mm -> 85.8 x 32.4 mm
