File: project/FSK/eagle/FSK/FSK.brd (EAGLE design)
At the start: 100 x 80 mm, 16 parts, among them X1 SMA-142-0711-821/826

Commit message: routed FSK test board
Parts:
- removed INPUT1, INPUT2, INPUT3, INPUT4: TEE_TL1, ECE532_Parts:TEE_TL1
- added 2.4FIL, 2.4TUNED, 2.6FIL, 2.6TUNED: TEE_TL1, ECE532_Parts:TEE_TL1
- added X2, X3, X4, X5: SMA-142-0711-821/826, con-coax:J502-ND-142-0711-821/826
- moved R1 195.9 mm to (111.6, 51.6), turned to 90 degrees
- moved U$2 191.8 mm to (107.2, 54.5), turned to 270 degrees
- moved C1 189.4 mm to (108.7, 52.5), turned to 270 degrees
- moved C2 184.4 mm to (109.2, 19.0), turned to 270 degrees
- moved R3 178.9 mm to (97.7, 54.5)
- moved U$3 157.8 mm to (107.6, 21.0), turned to 270 degrees
- moved R4 136.2 mm to (98.1, 21.0)
- moved R2 45.5 mm to (112.3, 18.2), turned to 90 degrees
- moved FILTER2 7.68 mm to (63.4, 21.1)
- moved FILTER1 7.30 mm to (63.2, 54.5)
- moved X1 1.57 mm to (-2.52, 37.8)
Connections:
- net N$1 renamed 2.4GHZ
- net N$2 renamed 2.6GHZ
- net 2.4FIL: now also 2.4FIL.T_B, 2.4FIL.T_L, 2.4FIL.T_R, FILTER1.OUT; no longer INPUT4.T_B, INPUT4.T_L, INPUT4.T_R
- net 2.4TUNED: now also 2.4TUNED.T_B, 2.4TUNED.T_L, 2.4TUNED.T_R; no longer INPUT3.T_B, INPUT3.T_L, INPUT3.T_R
- net 2.6FIL: now also 2.6FIL.T_B, 2.6FIL.T_L, 2.6FIL.T_R; no longer INPUT2.T_B, INPUT2.T_L, INPUT2.T_R
- net 2.6TUNED: now also 2.6TUNED.T_B, 2.6TUNED.T_L, 2.6TUNED.T_R; no longer INPUT1.T_B, INPUT1.T_L, INPUT1.T_R
Routing:
- net N$4: track 0.00 -> 4.12 mm
- net N$3: track 0.00 -> 3.77 mm
- added copper zone on layer 1, net 2.6FIL
- added copper zone on layer 1, net 2.6TUNED
- removed copper zone on layer 1, net INPUT4
- removed copper zone on layer 1, net INPUT5
- removed copper zone on layer 1, net INPUT7
- removed copper zone on layer 1, net INPUT8
Other:
- board size 100 x 80 mm -> 120 x 74 mm
- board text added: "2.4 GHz"
- board text added: "2.6 GHz"
- board text added: "W. Splitter"
- board text added: "test port"

Commit message: fixed FSK board
Routing:
- net 2.6GHZ: track 0.00 -> 9.87 mm
- net 2.4GHZ: track 0.00 -> 9.87 mm
- added copper zone on layer 1, net 2.4GHZ
- added copper zone on layer 1, net 2.6GHZ
