File: project/FSK/eagle/FSK/FSK.sch (EAGLE design)
At the start: 16 parts, among them X1 SMA-142-0711-821/826

Commit message: routed FSK test board
Parts:
- added X2, X3, X4, X5: SMA-142-0711-821/826, con-coax:SMA-142-0711-821/826
- renumbered INPUT1 to 2.6TUNED, INPUT2 to 2.6FIL, INPUT3 to 2.4TUNED, INPUT4 to 2.4FIL
Connections:
- net N$1 renamed 2.4GHZ
- net N$2 renamed 2.6GHZ
- net 2.4FIL: now also FILTER1.OUT
Changed lines of the file:
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@@
 <?xml version="1.0" encoding="utf-8"?>
 <!DOCTYPE eagle SYSTEM "eagle.dtd">
-<eagle version="7.5.0">
+<eagle version="6.5.0">
 <drawing>
 <settings>
@@
 <layers>
 <layer number="1" name="Top" color="4" fill="1" visible="no" active="no"/>
+<layer number="2" name="Route2" color="1" fill="3" visible="no" active="no"/>
+<layer number="3" name="Route3" color="4" fill="3" visible="no" active="no"/>
+<layer number="4" name="Route4" color="1" fill="4" visible="no" active="no"/>
+<layer number="5" name="Route5" color="4" fill="4" visible="no" active="no"/>
+<layer number="6" name="Route6" color="1" fill="8" visible="no" active="no"/>
+<layer number="7" name="Route7" color="4" fill="8" visible="no" active="no"/>
+<layer number="8" name="Route8" color="1" fill="2" visible="no" active="no"/>
+<layer number="9" name="Route9" color="4" fill="2" visible="no" active="no"/>
+<layer number="10" name="Route10" color="1" fill="7" visible="no" active="no"/>
+<layer number="11" name="Route11" color="4" fill="7" visible="no" active="no"/>
+<layer number="12" name="Route12" color="1" fill="5" visible="no" active="no"/>
+<layer number="13" name="Route13" color="4" fill="5" visible="no" active="no"/>
+<layer number="14" name="Route14" color="1" fill="6" visible="no" active="no"/>
+<layer number="15" name="Route15" color="4" fill="6" visible="no" active="no"/>
 <layer number="16" name="Bottom" color="1" fill="1" visible="no" active="no"/>
 <layer number="17" name="Pads" color="2" fill="1" visible="no" active="no"/>
@@
 <part name="SUPPLY4" library="supply2" deviceset="GND1" device=""/>
 <part name="SUPPLY5" library="supply2" deviceset="GND1" device=""/>
-<part name="INPUT1" library="ECE532_Parts" deviceset="TEE_TL1" device=""/>
-<part name="INPUT2" library="ECE532_Parts" deviceset="TEE_TL1" device=""/>
+<part name="2.6TUNED" library="ECE532_Parts" deviceset="TEE_TL1" device=""/>
+<part name="2.6FIL" library="ECE532_Parts" deviceset="TEE_TL1" device=""/>
 <part name="R4" library="rcl" deviceset="R-US_" device="R0603"/>
 <part name="X1" library="con-coax" deviceset="SMA-" device="142-0711-821/826"/>
@@
 <part name="SUPPLY1" library="supply2" deviceset="GND1" device=""/>
 <part name="SUPPLY2" library="supply2" deviceset="GND1" device=""/>
-<part name="INPUT3" library="ECE532_Parts" deviceset="TEE_TL1" device=""/>
-<part name="INPUT4" library="ECE532_Parts" deviceset="TEE_TL1" device=""/>
+<part name="2.4TUNED" library="ECE532_Parts" deviceset="TEE_TL1" device=""/>
+<part name="2.4FIL" library="ECE532_Parts" deviceset="TEE_TL1" device=""/>
 <part name="R3" library="rcl" deviceset="R-US_" device="R0603"/>
+<part name="X2" library="con-coax" deviceset="SMA-" device="142-0711-821/826"/>
+<part name="X3" library="con-coax" deviceset="SMA-" device="142-0711-821/826"/>
+<part name="X4" library="con-coax" deviceset="SMA-" device="142-0711-821/826"/>
+<part name="X5" library="con-coax" deviceset="SMA-" device="142-0711-821/826"/>
 </parts>
 <sheets>
@@
 <instance part="SUPPLY4" gate="G$1" x="236.22" y="111.76"/>
 <instance part="SUPPLY5" gate="G$1" x="251.46" y="109.22"/>
-<instance part="INPUT1" gate="G$1" x="210.82" y="124.46"/>
-<instance part="INPUT2" gate="G$1" x="177.8" y="124.46"/>
+<instance part="2.6TUNED" gate="G$1" x="210.82" y="124.46"/>
+<instance part="2.6FIL" gate="G$1" x="177.8" y="124.46"/>
 <instance part="R4" gate="G$1" x="193.04" y="124.46"/>
-<instance part="X1" gate="G1" x="60.96" y="139.7"/>
+<instance part="X1" gate="G1" x="60.96" y="139.7" smashed="yes">
+<attribute name="NAME" x="58.42" y="143.002" size="1.778" layer="95"/>
+</instance>
 <instance part="SUPPLY3" gate="G$1" x="63.5" y="129.54"/>
 <instance part="U$2" gate="G$1" x="223.52" y="152.4" smashed="yes"/>
@@
 <instance part="SUPPLY1" gate="G$1" x="236.22" y="139.7"/>
 <instance part="SUPPLY2" gate="G$1" x="251.46" y="137.16"/>
-<instance part="INPUT3" gate="G$1" x="210.82" y="152.4"/>
-<instance part="INPUT4" gate="G$1" x="177.8" y="152.4"/>
+<instance part="2.4TUNED" gate="G$1" x="210.82" y="152.4"/>
+<instance part="2.4FIL" gate="G$1" x="177.8" y="152.4"/>
 <instance part="R3" gate="G$1" x="193.04" y="152.4"/>
+<instance part="X2" gate="G1" x="96.52" y="177.8" smashed="yes" rot="R270">
+<attribute name="NAME" x="99.822" y="180.34" size="1.778" layer="95" rot="R270"/>
+</instance>
+<instance part="X3" gate="G1" x="96.52" y="99.06" smashed="yes" rot="R90">
+<attribute name="NAME" x="93.218" y="96.52" size="1.778" layer="95" rot="R90"/>
+</instance>
+<instance part="X4" gate="G1" x="160.02" y="99.06" smashed="yes" rot="R90">
+<attribute name="NAME" x="156.718" y="96.52" size="1.778" layer="95" rot="R90"/>
+</instance>
+<instance part="X5" gate="G1" x="160.02" y="177.8" smashed="yes" rot="R270">
+<attribute name="NAME" x="163.322" y="180.34" size="1.778" layer="95" rot="R270"/>
+</instance>
 </instances>
 <busses>
@@
 <net name="2.6FIL" class="0">
 <segment>
-<pinref part="INPUT2" gate="G$1" pin="T_B"/>
-<pinref part="INPUT2" gate="G$1" pin="T_L"/>
+<pinref part="2.6FIL" gate="G$1" pin="T_B"/>
+<pinref part="2.6FIL" gate="G$1" pin="T_L"/>
 <wire x1="170.18" y1="124.46" x2="167.64" y2="124.46" width="0.1524" layer="91"/>
 <wire x1="167.64" y1="124.46" x2="167.64" y2="116.84" width="0.1524" layer="91"/>
 <wire x1="167.64" y1="116.84" x2="177.8" y2="116.84" width="0.1524" layer="91"/>
 <wire x1="177.8" y1="116.84" x2="185.42" y2="116.84" width="0.1524" layer="91"/>
-<pinref part="INPUT2" gate="G$1" pin="T_R"/>
+<pinref part="2.6FIL" gate="G$1" pin="T_R"/>
 <pinref part="R4" gate="G$1" pin="1"/>
 <wire x1="185.42" y1="124.46" x2="187.96" y2="124.46" width="0.1524" layer="91"/>
@@
 <net name="2.6TUNED" class="0">
 <segment>
-<pinref part="INPUT1" gate="G$1" pin="T_R"/>
+<pinref part="2.6TUNED" gate="G$1" pin="T_R"/>
 <pinref part="U$3" gate="G$1" pin="A"/>
 <wire x1="218.44" y1="124.46" x2="220.98" y2="124.46" width="0.1524" layer="91"/>
-<pinref part="INPUT1" gate="G$1" pin="T_L"/>
-<pinref part="INPUT1" gate="G$1" pin="T_B"/>
+<pinref part="2.6TUNED" gate="G$1" pin="T_L"/>
+<pinref part="2.6TUNED" gate="G$1" pin="T_B"/>
 <wire x1="210.82" y1="116.84" x2="210.82" y2="114.3" width="0.1524" layer="91"/>
 <wire x1="210.82" y1="114.3" x2="203.2" y2="114.3" width="0.1524" layer="91"/>
@@
 </segment>
 </net>
-<net name="N$1" class="0">
+<net name="2.4GHZ" class="0">
 <segment>
 <pinref part="U$1" gate="G$1" pin="P$2"/>
@@
 </segment>
 </net>
-<net name="N$2" class="0">
+<net name="2.6GHZ" class="0">
 <segment>
 <pinref part="U$1" gate="G$1" pin="P$3"/>
@@
 <net name="2.4FIL" class="0">
 <segment>
-<pinref part="INPUT4" gate="G$1" pin="T_B"/>
-<pinref part="INPUT4" gate="G$1" pin="T_L"/>
+<pinref part="2.4FIL" gate="G$1" pin="T_B"/>
+<pinref part="2.4FIL" gate="G$1" pin="T_L"/>
 <wire x1="170.18" y1="152.4" x2="167.64" y2="152.4" width="0.1524" layer="91"/>
 <wire x1="167.64" y1="152.4" x2="167.64" y2="144.78" width="0.1524" layer="91"/>
 <wire x1="167.64" y1="144.78" x2="177.8" y2="144.78" width="0.1524" layer="91"/>
 <wire x1="177.8" y1="144.78" x2="185.42" y2="144.78" width="0.1524" layer="91"/>
-<pinref part="INPUT4" gate="G$1" pin="T_R"/>
+<pinref part="2.4FIL" gate="G$1" pin="T_R"/>
 <pinref part="R3" gate="G$1" pin="1"/>
 <wire x1="185.42" y1="152.4" x2="187.96" y2="152.4" width="0.1524" layer="91"/>
 <wire x1="185.42" y1="144.78" x2="185.42" y2="152.4" width="0.1524" layer="91"/>
-<wire x1="167.64" y1="152.4" x2="157.48" y2="152.4" width="0.1524" layer="91"/>
+<pinref part="FILTER1" gate="G$1" pin="OUT"/>
+<wire x1="157.48" y1="152.4" x2="167.64" y2="152.4" width="0.1524" layer="91"/>
 </segment>
 </net>
 <net name="2.4TUNED" class="0">
 <segment>
-<pinref part="INPUT3" gate="G$1" pin="T_R"/>
+<pinref part="2.4TUNED" gate="G$1" pin="T_R"/>
 <pinref part="U$2" gate="G$1" pin="A"/>
 <wire x1="218.44" y1="152.4" x2="220.98" y2="152.4" width="0.1524" layer="91"/>
-<pinref part="INPUT3" gate="G$1" pin="T_L"/>
-<pinref part="INPUT3" gate="G$1" pin="T_B"/>
+<pinref part="2.4TUNED" gate="G$1" pin="T_L"/>
+<pinref part="2.4TUNED" gate="G$1" pin="T_B"/>
 <wire x1="210.82" y1="144.78" x2="210.82" y2="142.24" width="0.1524" layer="91"/>
 <wire x1="210.82" y1="142.24" x2="203.2" y2="142.24" width="0.1524" layer="91"/>

Commit message: fixed FSK board
Changed lines of the file:
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@@
-</segment>
-</net>
-<net name="2.4GHZ" class="0">
-<segment>
-<pinref part="U$1" gate="G$1" pin="P$2"/>
-<wire x1="91.44" y1="142.24" x2="91.44" y2="152.4" width="0.1524" layer="91"/>
-<pinref part="FILTER1" gate="G$1" pin="IN"/>
-<wire x1="91.44" y1="152.4" x2="106.68" y2="152.4" width="0.1524" layer="91"/>
-</segment>
-</net>
-<net name="2.6GHZ" class="0">
-<segment>
-<pinref part="U$1" gate="G$1" pin="P$3"/>
-<wire x1="91.44" y1="137.16" x2="91.44" y2="124.46" width="0.1524" layer="91"/>
-<pinref part="FILTER2" gate="G$1" pin="IN"/>
-<wire x1="91.44" y1="124.46" x2="106.68" y2="124.46" width="0.1524" layer="91"/>
 </segment>
 </net>
@@
 </segment>
 </net>
+<net name="2.4GHZ" class="0">
+<segment>
+<pinref part="U$1" gate="G$1" pin="P$2"/>
+<pinref part="FILTER1" gate="G$1" pin="IN"/>
+<wire x1="91.44" y1="142.24" x2="106.68" y2="142.24" width="0.1524" layer="91"/>
+<wire x1="106.68" y1="142.24" x2="106.68" y2="152.4" width="0.1524" layer="91"/>
+</segment>
+</net>
+<net name="2.6GHZ" class="0">
+<segment>
+<pinref part="U$1" gate="G$1" pin="P$3"/>
+<pinref part="FILTER2" gate="G$1" pin="IN"/>
+<wire x1="91.44" y1="137.16" x2="106.68" y2="137.16" width="0.1524" layer="91"/>
+<wire x1="106.68" y1="137.16" x2="106.68" y2="124.46" width="0.1524" layer="91"/>
+</segment>
+</net>
