File: project/FSK/eagle/Untitled.sch (EAGLE design)
At the start: 9 parts, among them IC1 74AUC1G32DCK

Commit message: added FSK version 2
Parts:
- added R6: 10k, rcl:R-US_R1206
- R1: value 4.7k -> 10k
Connections:
- new net N$10: R2.2, R4.2, U$2.REF
- new net N$11: LED1.C, U$1.C
- new net N$12: LED1.B, U$1.B
- new net N$13: LED1.A, U$1.A
- new net N$14: LED1.G, U$1.G
- new net N$15: LED1.F, U$1.F
- new net N$8: LED1.E, U$1.E
- new net N$9: LED1.D, U$1.D
- net AGND: now also LED1.C@1, LED1.C@2, R6.1
- net N$2: now also U$1.LT; no longer U$1.BL
- net N$3: now also R6.2, U$1.BL; no longer U$1.LT
- net VCC: no longer R2.2, R4.2
Other:
- moved on the sheet: R2, R3, R4, R5
